File: ORA_ControlBoard/ORA_ControlBoard-main_Rev2/ORA_ControlBoard-main_Rev2.kicad_pcb (KiCad board)
At the start: 2 copper layers, 100 x 60 mm, 72 parts, among them J1 SM04B-GHS-TB, J2 Conn_01x04_Pin, J3 USB_B_Micro, J4 12V, J5 SM04B-GHS-TB, J6 Conn_02x03_Top_Bottom, J7 Conn_01x05_Pin, J8 Conn_01x05_Pin, J9 Stack Light, Q1 BS170, Q2 IRF9540N, Q3 BS170, Q4 IRF9540N, Q5 BS170, Q6 IRF9540N, SW1 Reset, U1 ATmega32U4-A, U2 MCP25625-x-SS, U5 NCP1117-5.0_SOT223, U6 IMU_MOUNT, Y1 8Mhz, Y2 16MHz

Commit message: Fixed Spring Cleaning
Other:
- board text added: "ORA IGVC 2023/24 Zenith Rev 2"
- board text removed: "ORA IGVC 2023/24 Control Board REV 1"
Changed lines of the file:
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@@
 		(layer "Edge.Cuts")
 	)
-	(gr_text "ORA IGVC 2023/24 Control Board REV 1"
+	(gr_text "ORA IGVC 2023/24 Zenith Rev 2\n"
 		(at 181.6 95.8 0)
 		(layer "B.SilkS")

Commit message: le testing
Other:
- board text added: "3/11/2024"
- board text removed: "1/10/2024"
Changed lines of the file:
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@@
 		)
 	)
-	(gr_text "1/10/2024\n"
+	(gr_text "3/11/2024\n"
 		(at 170.1 97.7 0)
 		(layer "B.SilkS")

Commit message: "Final" Rev 2 changes
Parts:
- removed the C1 at (171.0, 78.0)
- removed the C1 at (180.3, 59.8)
- removed the C2 at (171.0, 74.0)
- removed the C2 at (177.8, 59.8)
- removed D5: IMU_LED, LED_SMD:LED_0805_2012Metric_Pad1.15x1.40mm_HandSolder
- removed Q2, Q4, Q6: IRF9540N, Package_TO_SOT_THT:TO-220-3_Vertical
- removed R7: 470, Resistor_SMD:R_0805_2012Metric_Pad1.20x1.40mm_HandSolder
- added C1: 22pF, Capacitor_SMD:C_0805_2012Metric_Pad1.18x1.45mm_HandSolder, F.Cu at (177.1, 72.6)
- added C2: 22pF, Capacitor_SMD:C_0805_2012Metric_Pad1.18x1.45mm_HandSolder, F.Cu at (174.1, 72.6)
- added G***: LOGO, AdditionalParts:ORA_Logo_V2, F.Cu at (106.8, 87.7)
- J3: footprint Connector_USB:USB_Micro-B_Amphenol_10118193-0002LF_Horizontal -> AdditionalParts:AMPHENOL_10118192-0002LF
- J6: moved to B.Cu
- TR1: renamed from R1; moved to B.Cu
- moved J2 51.6 mm to (92.5, 83.7)
- moved J1 44.7 mm to (187.3, 65.0), turned to 90 degrees
- moved J5 41.9 mm to (187.3, 79.0), turned to 90 degrees
- moved Q1 29.5 mm to (142.0, 96.7)
- moved R15 29.5 mm to (146.0, 99.8)
- moved R16 29.5 mm to (146.0, 95.8)
- moved R14 23.9 mm to (141.0, 93.7), turned to 0 degrees
- moved TR1 21.4 mm to (161.8, 88.8)
- moved R22 21.1 mm to (119.0, 94.0), turned to 0 degrees
- moved Q5 17.2 mm to (120.0, 96.7)
- moved R20 17.2 mm to (124.0, 96.0)
- moved R21 17.2 mm to (124.0, 100.0)
- moved Y1 15.5 mm to (173.1, 77.6), turned to 0 degrees
- moved J7 14.9 mm to (102.5, 100.0), turned to 90 degrees
- moved R1 14.1 mm to (175.6, 82.1), turned to 0 degrees
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Connections:
- C7 pad 1: VBUS -> +5V
- F1 pad 1: VBUS -> +5V
- J9 pad 1: GND -> PWRIN
- J9 pad 2: LED_G -> LED_R
- J9 pad 3: LED_Y -> LED_G
- J9 pad 4: LED_R -> LED_B
- R14 pad 1: PWRIN -> LED_R
- R17 pad 1: LEDPWR_Y -> LEDPWR_G
- R19 pad 1: PWRIN -> LED_G
- R20 pad 1: LEDPWR_G -> LEDPWR_B
- R22 pad 1: PWRIN -> LED_B
- U1 pad 26: LEDPWR_Y -> LEDPWR_G
- U1 pad 27: LEDPWR_G -> LEDPWR_B
- U1 pad 7: VBUS -> +5V
Routing:
- net +5V: track 168.9 -> 297.5 mm, vias 8 -> 12
- net CAN_CS: track 0.00 -> 83.4 mm, vias 0 -> 2
- net CAN_SO: track 44.3 -> 119.6 mm, vias 1 -> 3
- net CAN_SCK: track 25.2 -> 91.9 mm, vias 1 -> 4
- net CAN_SI: track 46.9 -> 112.2 mm, vias 1 -> 4
- net CAN_INT: track 0.00 -> 60.7 mm
- net CAN_H: track 6.12 -> 45.0 mm, vias 0 -> 1
- net CAN_L: track 8.34 -> 43.7 mm, vias 0 -> 3
- net LED_Y: track 35.3 -> 0.00 mm, vias 2 -> 0
- net LED_R: track 23.1 -> 56.4 mm
- net LED_B: track 0.00 -> 29.3 mm, vias 0 -> 1
- net VBUS: track 26.6 -> 0.00 mm, vias 2 -> 0
- net LEDPWR_Y: track 26.0 -> 0.00 mm
- net Net-(D3-A): track 12.2 -> 34.5 mm, vias 0 -> 2
- net LEDPWR_B: track 0.00 -> 18.6 mm, vias 0 -> 2
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Other:
- board size 100 x 60 mm -> 100 x 52.5 mm
- board text added: "ORA IGVC 2023/24 Control Board REV 2"
- board text added: "Robotics Association of Oakland University"
- board text removed: "H"
- board text removed: "L"
- board text removed: "ORA IGVC 2023/24 Zenith Rev 2"
